File: PCB/Hackboard_v1.kicad_pcb (KiCad board)
At the start: 2 copper layers, 76.2 x 99.5 mm, 26 parts, among them SW1 SW_Push, SW10 RotaryEncoder_Switch, SW2 SW_Push, SW3 SW_Push, SW4 SW_Push, SW5 SW_Push, SW6 SW_Push, SW7 SW_Push, SW8 SW_Push, SW9 SW_Push, U1 MOUDLE-SEEEDUINO-XIAO, U2 ER_OLEDM0.91_1x-I2C

Commit message: ww
Connections:
- D10 pad 1: (no net) -> Net-(D10-K)
- D2 pad 1: (no net) -> Net-(D2-K)
- D3 pad 1: (no net) -> Net-(D3-K)
- D4 pad 1: (no net) -> Net-(D4-K)
- D5 pad 1: (no net) -> Net-(D5-K)
- D6 pad 1: (no net) -> Net-(D6-K)
- D7 pad 1: (no net) -> Net-(D7-K)
- D8 pad 1: (no net) -> Net-(D8-K)
- D9 pad 1: (no net) -> Net-(D9-K)
Routing:
- net Net-(D8-K): track 0.00 -> 15.1 mm, vias 0 -> 1
- net Net-(D2-K): track 0.00 -> 12.4 mm, vias 0 -> 2
- net Net-(D4-K): track 0.00 -> 11.0 mm
- net Net-(D9-K): track 0.00 -> 8.98 mm
- net Net-(D3-K): track 0.00 -> 8.31 mm, vias 0 -> 2
- net Net-(D7-K): track 0.00 -> 7.93 mm
- net Net-(D6-K): track 0.00 -> 7.40 mm
- net Net-(D5-K): track 0.00 -> 6.81 mm, vias 0 -> 1
- net Net-(D10-K): track 0.00 -> 6.35 mm
